Commit message: try diff_drive_ontroller

File: src/orange_robot/urdf/orange.urdf (robot description, URDF)
Before this commit: robot orange_robot, 6 links, 5 joints
Joints:
- removed joint base_to_left_wheel
- removed joint base_to_right_wheel
- added joint wheel_left_joint: type fixed, parent base_link, child left_wheel, origin xyz=0 0.145 0.032 rpy=-1.57 0 0
- added joint wheel_right_joint: type fixed, parent base_link, child right_wheel, origin xyz=0 -0.145 0.032 rpy=1.57 0 0

Commit message: run with ros_control

File: src/orange_robot/urdf/orange.urdf (robot description, URDF)
Before this commit: robot orange_robot, 6 links, 5 joints
Links:
- removed link left_wheel
- removed link right_wheel
- added link wheel_left_link; collision cylinder length=0.023 radius=0.068; visual cylinder length=0.023 radius=0.068
- added link wheel_right_link; collision cylinder length=0.023 radius=0.068; visual cylinder length=0.023 radius=0.068
Joints:
- joint wheel_left_joint: axis (none) -> 0 0 1; child left_wheel -> wheel_left_link; type fixed -> continuous
- joint wheel_right_joint: axis (none) -> 0 0 -1; child right_wheel -> wheel_right_link; type fixed -> continuous
